File: compute-board.kicad_pcb (KiCad board)
At the start: 4 copper layers, 70 x 70 mm, 5 parts, among them J1 PC104

Commit message: Initial commit
Parts:
- added C1: 100nF, Capacitor_SMD:C_1206_3216Metric_Pad1.33x1.80mm_HandSolder, F.Cu at (99.2, 91.7)
- added C10: 2.2uF, Capacitor_SMD:C_1206_3216Metric_Pad1.33x1.80mm_HandSolder, F.Cu at (101.9, 55.1)
- added C11: 2.2uF, Capacitor_SMD:C_1206_3216Metric_Pad1.33x1.80mm_HandSolder, F.Cu at (101.9, 58.5)
- added C2: 22uF, Capacitor_Tantalum_SMD:CP_EIA-3528-21_Kemet-B_HandSolder, F.Cu at (93.6, 88.6)
- added C3: 10uF, Capacitor_SMD:C_1206_3216Metric_Pad1.33x1.80mm_HandSolder, F.Cu at (129.0, 77.0)
- added C4: 4.7uF, Capacitor_SMD:C_1206_3216Metric_Pad1.33x1.80mm_HandSolder, F.Cu at (138.7, 78.2)
- added C5: 1uF, Capacitor_SMD:C_1206_3216Metric_Pad1.33x1.80mm_HandSolder, F.Cu at (116.4, 87.8)
- added C6: 10uF, Capacitor_SMD:C_1206_3216Metric_Pad1.33x1.80mm_HandSolder, F.Cu at (121.2, 76.9)
- added C7: 1uF, Capacitor_SMD:C_1206_3216Metric_Pad1.33x1.80mm_HandSolder, F.Cu at (146.2, 96.9)
- added C8: 4.7uF, Capacitor_SMD:C_1206_3216Metric_Pad1.33x1.80mm_HandSolder, F.Cu at (127.4, 86.7)
- added C9: 0.1uF, Capacitor_SMD:C_1206_3216Metric_Pad1.33x1.80mm_HandSolder, F.Cu at (101.9, 51.8)
- added D1: WS2812B-2020, LED_SMD:LED_WS2812B-2020_PLCC4_2.0x2.0mm, F.Cu at (104.4, 97.0)
- added G***: LOGO, LOGO:logo, F.Cu at (94.5, 42.6)
- added G***: LOGO, LOGO:logo, B.Cu at (94.9, 42.3)
- added J2: ESP_PROG, TestPoint:TestPoint_Pad_2.0x2.0mm, F.Cu at (131.0, 92.8)
- added J3: ESP_PROGRAM, Connector_JST:JST_XH_B4B-XH-AM_1x04_P2.50mm_Vertical, F.Cu at (153.4, 71.4)
- added J4: i2c, Connector_JST:JST_XH_B4B-XH-AM_1x04_P2.50mm_Vertical, F.Cu at (153.3, 86.8)
- added J5: 104031-0811, Project-Specific:1040310811, B.Cu at (103.1, 55.2)
- added J6: RST, TestPoint:TestPoint_Pad_2.0x2.0mm, F.Cu at (121.0, 90.3)
- added R1: 50k, Resistor_SMD:R_1206_3216Metric_Pad1.30x1.75mm_HandSolder, F.Cu at (94.4, 50.2)
- added R2: 50k, Resistor_SMD:R_1206_3216Metric_Pad1.30x1.75mm_HandSolder, F.Cu at (94.4, 53.5)
- added R3: 50k, Resistor_SMD:R_1206_3216Metric_Pad1.30x1.75mm_HandSolder, F.Cu at (94.4, 56.8)
- added R4: 50k, Resistor_SMD:R_1206_3216Metric_Pad1.30x1.75mm_HandSolder, F.Cu at (94.4, 60.1)
- added R5: 2.2K, Resistor_SMD:R_1206_3216Metric_Pad1.30x1.75mm_HandSolder, F.Cu at (138.7, 74.2)
- added R6: 2.2K, Resistor_SMD:R_1206_3216Metric_Pad1.30x1.75mm_HandSolder, F.Cu at (138.8, 71.4)
- added R7: 10K, Resistor_SMD:R_1206_3216Metric_Pad1.30x1.75mm_HandSolder, F.Cu at (112.7, 87.8)
- added R8: 10K, Resistor_SMD:R_1206_3216Metric_Pad1.30x1.75mm_HandSolder, F.Cu at (146.2, 93.7)
- added RESET1: RESET, Button_Switch_SMD:SW_Push_1P1T_XKB_TS-1187A, F.Cu at (112.5, 95.5)
- added SW1: ESP Program, Button_Switch_SMD:SW_Push_1P1T_XKB_TS-1187A, F.Cu at (125.1, 95.5)
- added SW2: WEB_CONF, Button_Switch_SMD:SW_Push_1P1T_XKB_TS-1187A, F.Cu at (137.2, 95.4)
- added U1: ESP32-WROOM-32E, RF_Module:ESP32-WROOM-32D, F.Cu at (99.5, 75.4)
- added U2: XC6220B331MR, Package_TO_SOT_SMD:SOT-23-5, F.Cu at (133.4, 81.5)
- added U3: TPS3839DBZ, Package_TO_SOT_SMD:SOT-23, F.Cu at (115.4, 82.0)
- added U4: XC6220B331MR, Package_TO_SOT_SMD:SOT-23-5, F.Cu at (124.8, 82.1)
- added V_BAT1: Conn_01x02, TerminalBlock_Altech:Altech_AK300_1x02_P5.00mm_45-Degree, F.Cu at (150.7, 55.0)
Connections:
- J1 pad 14: GPIO12 -> CONFIG_ENA
- J1 pad 16: GPIO13 -> VCC_AUX_ENA
- J1 pad 23: GPIO15 -> LED1
- J1 pad 25: GPIO0 -> ESP_PROG
- J1 pad 29: GPIO05 -> GPIO05/SD_CS
- J1 pad 30: GPIO18 -> GPIO18/SD_SCK
- J1 pad 31: GPIO19 -> GPIO19/SD_MISO
- J1 pad 33: GPIO21 -> SDA
- J1 pad 36: GPIO22 -> SCL
- J1 pad 37: GPIO23 -> GPIO23/SD_MOSI
- J1 pad 39: AUX08 -> GND
- J1 pad 40: AUX09 -> V_BAT
Routing:
- net ESP_PROG: track 0.00 -> 112.0 mm, vias 0 -> 3
- net VCC: track 0.00 -> 111.9 mm, vias 0 -> 5
- net CONFIG_ENA: track 0.00 -> 111.6 mm, vias 0 -> 2
- net RXD0: track 0.00 -> 110.4 mm, vias 0 -> 2
- net SCL: track 0.00 -> 108.5 mm, vias 0 -> 2
- net V_BAT: track 0.00 -> 100.1 mm, vias 0 -> 1
- net GPIO23/SD_MOSI: track 0.00 -> 99.4 mm, vias 0 -> 1
- net TXD0: track 0.00 -> 99.1 mm, vias 0 -> 1
- net SDA: track 0.00 -> 98.2 mm, vias 0 -> 3
- net GPIO19/SD_MISO: track 0.00 -> 94.4 mm, vias 0 -> 2
- net GPIO05/SD_CS: track 0.00 -> 90.7 mm, vias 0 -> 2
- net GPIO18/SD_SCK: track 0.00 -> 88.8 mm, vias 0 -> 1
- net VCC_AUX_ENA: track 0.00 -> 81.4 mm, vias 0 -> 2
- net LED1: track 0.00 -> 77.6 mm, vias 0 -> 3
- net GPIO32: track 0.00 -> 55.5 mm, vias 0 -> 1
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- added copper zone on B.Cu, net GND
- added copper zone on F.Cu, net GND
- added copper zone on In1.Cu, net GND
- added copper zone on In2.Cu, net VCC_AUX
Other:
- board text added: "AUX01"
- board text added: "AUX02"
- board text added: "AUX03"
- board text added: "AUX04"
- board text added: "AUX05"
- board text added: "AUX06"
- board text added: "AUX07"
- board text added: "CFG_ENA"
- board text added: "COMPUTE BOARD V1.0.0 JAN/2026 VA7RCV"
- board text added: "CONF"
- board text added: "DATA"
- board text added: "ESP_PROG"
- board text added: "GND"
- board text added: "GPIO02"
- board text added: "GPIO04"
- board text added: "GPIO05/SD_CS"
- board text added: "GPIO14"
- board text added: "GPIO16"
- board text added: "GPIO17"
- board text added: "GPIO18/SD_SCK"
- board text added: "GPIO19/SD_MISO"
- board text added: "GPIO23/SD_MOSI"
- board text added: "GPIO25"
- board text added: "GPIO26"
- board text added: "GPIO27"
- board text added: "GPIO32"
- board text added: "GPIO33"
- board text added: "GPIO34"
- board text added: "GPIO36"
- board text added: "GPIO39"
- board text added: "I2C"
- board text added: "LED1"
- board text added: "MICRO SD"
- board text added: "PROG"
- board text added: "PROGRAM"
- board text added: "RESET"
- board text added: "RXD0"
- board text added: "SCL"
- board text added: "SDA"
- board text added: "TXD0"
- board text added: "VCC"
- board text added: "VCC_AUX"
- board text added: "V_AUX"
- board text added: "V_A_ENA"
- board text added: "V_BAT"
- board text added: "https://jesus.identitylabs.mx"

Commit message: FIX: routing recommendations
Parts:
- moved C6 7.33 mm to (128.2, 78.9)
- moved C3 3.17 mm to (132.0, 75.9)
Routing:
- net VCC_AUX_ENA: track 81.4 -> 74.6 mm
- net V_BAT: track 100.1 -> 94.4 mm
- net VCC: track 111.9 -> 108.2 mm, vias 5 -> 4
- net GPIO19/SD_MISO: track 94.4 -> 92.4 mm
- net GPIO18/SD_SCK: track 88.8 -> 87.9 mm
- net GPIO23/SD_MOSI: track 99.4 -> 98.6 mm, vias 1 -> 2
- net GPIO05/SD_CS: track 90.7 -> 90.2 mm
- net GND: vias 173 -> 198
- net (no net): vias 9 -> 0

Commit message: UPDATE: schematic and pcb revision
Other:
- board text added: "COMPUTE BOARD V1.0.1 APRIL/2026 VA7RCV"
- board text removed: "COMPUTE BOARD V1.0.0 JAN/2026 VA7RCV"
Changed lines of the file:
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@@
 		)
 	)
-	(gr_text "COMPUTE BOARD V1.0.0\nJAN/2026\nVA7RCV"
+	(gr_text "COMPUTE BOARD V1.0.1\nAPRIL/2026\nVA7RCV"
 		(at 150.092893 97.892893 0)
 		(layer "B.SilkS")
