File: compute-board.kicad_pcb (KiCad board)
At the start: 4 copper layers, 70 x 70 mm, 40 parts, among them J1 PC104, J2 ESP_PROG, J3 ESP_PROGRAM, J4 i2c, J5 104031-0811, J6 RST, SW1 ESP Program, SW2 WEB_CONF, U1 ESP32-WROOM-32E, U2 XC6220B331MR, U3 TPS3839DBZ, U4 XC6220B331MR

Commit message: (fix): various hardware designgs issues.
1. Add thermal reliefs.
2. Remove Pullup on CONFIG button, this was causing the esp32 to select
   1.8v FLASH.
3. Replace addresable led with a single color led.
Parts:
- removed C7: 1uF, Capacitor_SMD:C_1206_3216Metric_Pad1.33x1.80mm_HandSolder
- removed D1: WS2812B-2020, LED_SMD:LED_WS2812B-2020_PLCC4_2.0x2.0mm
- added D2: LED, LED_SMD:LED_0603_1608Metric_Pad1.05x0.95mm_HandSolder, F.Cu at (103.5, 97.6)
- R8: value 10K -> 1K
- moved R8 42.9 mm to (103.4, 95.2), turned to 0 degrees
Connections:
- R8 pad 1: VCC_AUX -> Net-(D2-K)
- R8 pad 2: CONFIG_ENA -> GND
Routing:
- net CONFIG_ENA: track 111.6 -> 103.8 mm
- net VCC_AUX: track 29.2 -> 26.0 mm, vias 13 -> 11
- net Net-(D2-K): track 0.00 -> 2.74 mm
- net LED1: track 77.6 -> 78.6 mm
- net GND: vias 198 -> 200
Other:
- board text added: "COMPUTE BOARD V1.1.0 JULY/2026 VA7RCV"
- board text removed: "COMPUTE BOARD V1.0.1 APRIL/2026 VA7RCV"
- board text removed: "DATA"
